File: keyboard.kicad_pcb (KiCad board)
At the start: 2 copper layers, 322 x 134.5 mm, 174 parts, among them SW1 SW_Push, SW10 SW_Push, SW11 SW_Push, SW12 SW_Push, SW13 SW_Push, SW14 SW_Push, SW15 SW_Push, SW16 SW_Push, SW17 SW_Push, SW18 SW_Push, SW19 SW_Push, SW2 SW_Push, SW20 SW_Push, SW21 SW_Push, SW22 SW_Push, SW23 SW_Push, SW24 SW_Push, SW25 SW_Push, SW26 SW_Push, SW27 SW_Push, SW28 SW_Push, SW29 SW_Push, SW3 SW_Push, SW30 SW_Push, SW31 SW_Push, SW32 SW_Push, SW33 SW_Push, SW34 SW_Push, SW35 SW_Push, SW36 SW_Push, SW37 SW_Push, SW38 SW_Push, SW39 SW_Push, SW4 SW_Push, SW40 SW_Push, SW41 SW_Push, SW42 SW_Push, SW43 SW_Push, SW44 SW_Push, SW45 SW_Push, SW46 SW_Push, SW47 SW_Push, SW48 SW_Push, SW49 SW_Push, SW5 SW_Push, SW50 SW_Push, SW51 SW_Push, SW52 SW_Push, SW53 SW_Push, SW54 SW_Push, SW55 SW_Push, SW56 SW_Push, SW57 SW_Push, SW58 SW_Push, SW59 SW_Push, SW6 SW_Push, SW60 SW_Push, SW61 SW_Push, SW62 SW_Push, SW63 SW_Push, SW64 SW_Push, SW65 SW_Push, SW66 SW_Push, SW67 SW_Push, SW68 SW_Push, SW69 SW_Push, SW7 SW_Push, SW70 SW_Push, SW71 SW_Push, SW72 SW_Push, SW73 SW_Push, SW74 SW_Push, SW75 SW_Push, SW76 SW_Push, SW77 SW_Push, SW78 SW_Push, SW79 SW_Push, SW8 SW_Push, SW80 SW_Push, SW81 SW_Push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

Commit message: Add files via upload
Parts:
- removed D83: 1N4148, Diode_THT:D_DO-35_SOD27_P7.62mm_Horizontal
Connections:
- A1 pad 31: unconnected-(A1-GPIO26_ADC0-Pad31) -> Net-(A1-GPIO26_ADC0)
- A1 pad 32: unconnected-(A1-GPIO27_ADC1-Pad32) -> Net-(A1-GPIO27_ADC1)
- SWENC_1 pad A: Net-(A1-GPIO5) -> Net-(A1-GPIO26_ADC0)
- SWENC_1 pad B: Net-(A1-GPIO4) -> Net-(A1-GPIO27_ADC1)
- SWENC_1 pad C: Net-(D83-A) -> Net-(U1-GND)
Routing:
- net Net-(A1-GPIO27_ADC1): track 0.00 -> 97.7 mm, vias 0 -> 1
- net Net-(A1-GPIO26_ADC0): track 0.00 -> 92.1 mm, vias 0 -> 1
- net Net-(A1-GPIO5): track 382.0 -> 299.0 mm, vias 1 -> 0
- net Net-(U1-GND): track 18.0 -> 71.9 mm
- net Net-(A1-GPIO4): track 433.7 -> 406.1 mm
- net Net-(D83-A): track 23.8 -> 0.00 mm
- net Net-(A1-GPIO21): track 403.0 -> 399.4 mm
Other:
- board text added: "600161.xyz"
- board text added: "designed and handbuilt by ttt"
