File: keyboard.kicad_sch (KiCad schematic)
At the start: 174 parts, among them SW1 SW_Push, SW10 SW_Push, SW11 SW_Push, SW12 SW_Push, SW13 SW_Push, SW14 SW_Push, SW15 SW_Push, SW16 SW_Push, SW17 SW_Push, SW18 SW_Push, SW19 SW_Push, SW2 SW_Push, SW20 SW_Push, SW21 SW_Push, SW22 SW_Push, SW23 SW_Push, SW24 SW_Push, SW25 SW_Push, SW26 SW_Push, SW27 SW_Push, SW28 SW_Push, SW29 SW_Push, SW3 SW_Push, SW30 SW_Push, SW31 SW_Push, SW32 SW_Push, SW33 SW_Push, SW34 SW_Push, SW35 SW_Push, SW36 SW_Push, SW37 SW_Push, SW38 SW_Push, SW39 SW_Push, SW4 SW_Push, SW40 SW_Push, SW41 SW_Push, SW42 SW_Push, SW43 SW_Push, SW44 SW_Push, SW45 SW_Push, SW46 SW_Push, SW47 SW_Push, SW48 SW_Push, SW49 SW_Push, SW5 SW_Push, SW50 SW_Push, SW51 SW_Push, SW52 SW_Push, SW53 SW_Push, SW54 SW_Push, SW55 SW_Push, SW56 SW_Push, SW57 SW_Push, SW58 SW_Push, SW59 SW_Push, SW6 SW_Push, SW60 SW_Push, SW61 SW_Push, SW62 SW_Push, SW63 SW_Push, SW64 SW_Push, SW65 SW_Push, SW66 SW_Push, SW67 SW_Push, SW68 SW_Push, SW69 SW_Push, SW7 SW_Push, SW70 SW_Push, SW71 SW_Push, SW72 SW_Push, SW73 SW_Push, SW74 SW_Push, SW75 SW_Push, SW76 SW_Push, SW77 SW_Push, SW78 SW_Push, SW79 SW_Push, SW8 SW_Push, SW80 SW_Push, SW81 SW_Push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

Commit message: Add files via upload
Parts:
- removed D83: 1N4148, Diode_THT:D_DO-35_SOD27_P7.62mm_Horizontal, symbol Diode:1N4148
Connections:
- net at A1.6 (GPIO4), SW20.1, SW34.1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: no longer SWENC_1.B
- net at A1.7 (GPIO5), SW21.1, SW35.1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: no longer SWENC_1.A
- net at SWENC_1.C: now also A1.13 (GND), A1.18 (GND), A1.23 (GND), A1.28 (GND), A1.3 (GND), A1.38 (GND), A1.8 (GND), U1.1 (GND)
- net at A1.31 (GPIO26_ADC0): now also SWENC_1.A
- net at A1.32 (GPIO27_ADC1): now also SWENC_1.B
Changed lines of the file:
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@@
 	)
 	(junction
-		(at 86.36 158.75)
-		(diameter 0)
-		(color 0 0 0 0)
-	)
-	(junction
 		(at 201.93 77.47)
 		(diameter 0)
@@
 	)
 	(junction
-		(at 97.79 161.29)
-		(diameter 0)
-		(color 0 0 0 0)
-	)
-	(junction
 		(at 167.64 40.64)
 		(diameter 0)
@@
 	)
 	(junction
+		(at 243.84 199.39)
+		(diameter 0)
+		(color 0 0 0 0)
+	)
+	(junction
 		(at 144.78 95.25)
 		(diameter 0)
@@
 	)
 	(junction
-		(at 135.89 118.11)
-		(diameter 0)
-		(color 0 0 0 0)
-	)
-	(junction
 		(at 73.66 48.26)
 		(diameter 0)
@@
 	(wire
 		(pts
+			(xy 285.75 203.2) (xy 146.05 203.2)
+		)
+		(stroke
+			(width 0)
+			(type default)
+		)
+	)
+	(wire
+		(pts
 			(xy 133.35 95.25) (xy 133.35 168.91)
 		)
@@
 	(wire
 		(pts
+			(xy 146.05 203.2) (xy 146.05 184.15)
+		)
+		(stroke
+			(width 0)
+			(type default)
+		)
+	)
+	(wire
+		(pts
 			(xy 63.5 8.89) (xy 63.5 22.86)
 		)
@@
 	(wire
 		(pts
+			(xy 147.32 204.47) (xy 273.05 204.47)
+		)
+		(stroke
+			(width 0)
+			(type default)
+		)
+	)
+	(wire
+		(pts
 			(xy 74.93 95.25) (xy 74.93 156.21)
 		)
@@
 	(wire
 		(pts
-			(xy 135.89 186.69) (xy 147.32 186.69)
+			(xy 243.84 205.74) (xy 243.84 199.39)
 		)
 		(stroke
@@
 	(wire
 		(pts
-			(xy 96.52 66.04) (xy 107.95 66.04)
+			(xy 144.78 186.69) (xy 144.78 205.74)
 		)
 		(stroke
@@
 	(wire
 		(pts
-			(xy 86.36 189.23) (xy 86.36 158.75)
+			(xy 266.7 176.53) (xy 285.75 176.53)
 		)
 		(stroke
@@
 	(wire
 		(pts
-			(xy 147.32 189.23) (xy 86.36 189.23)
+			(xy 96.52 66.04) (xy 107.95 66.04)
 		)
 		(stroke
@@
 	(wire
 		(pts
+			(xy 273.05 179.07) (xy 266.7 179.07)
+		)
+		(stroke
+			(width 0)
+			(type default)
+		)
+	)
+	(wire
+		(pts
 			(xy 133.35 77.47) (xy 133.35 95.25)
 		)
@@
 	(wire
 		(pts
+			(xy 285.75 176.53) (xy 285.75 203.2)
+		)
+		(stroke
+			(width 0)
+			(type default)
+		)
+	)
+	(wire
+		(pts
 			(xy 271.78 161.29) (xy 266.7 161.29)
 		)
@@
 	(wire
 		(pts
-			(xy 179.07 8.89) (xy 179.07 22.86)
+			(xy 147.32 186.69) (xy 144.78 186.69)
 		)
 		(stroke
@@
 	(wire
 		(pts
-			(xy 52.07 151.13) (xy 220.98 151.13)
+			(xy 179.07 8.89) (xy 179.07 22.86)
 		)
 		(stroke
@@
 	(wire
 		(pts
-			(xy 212.09 30.48) (xy 266.7 30.48)
+			(xy 52.07 151.13) (xy 220.98 151.13)
 		)
 		(stroke
@@
 	(wire
 		(pts
-			(xy 73.66 85.09) (xy 85.09 85.09)
+			(xy 212.09 30.48) (xy 266.7 30.48)
 		)
 		(stroke
@@
 	(wire
 		(pts
-			(xy 135.89 125.73) (xy 135.89 186.69)
+			(xy 73.66 85.09) (xy 85.09 85.09)
 		)
 		(stroke
@@
 	(wire
 		(pts
-			(xy 62.23 30.48) (xy 73.66 30.48)
+			(xy 144.78 205.74) (xy 243.84 205.74)
 		)
 		(stroke
@@
 	(wire
 		(pts
-			(xy 154.94 85.09) (xy 166.37 85.09)
+			(xy 62.23 30.48) (xy 73.66 30.48)
 		)
 		(stroke
@@
 	(wire
 		(pts
-			(xy 189.23 85.09) (xy 212.09 85.09)
+			(xy 154.94 85.09) (xy 166.37 85.09)
 		)
 		(stroke
@@
 	(wire
 		(pts
-			(xy 119.38 85.09) (xy 130.81 85.09)
+			(xy 189.23 85.09) (xy 212.09 85.09)
 		)
 		(stroke
@@
 	(wire
 		(pts
-			(xy 201.93 58.42) (xy 201.93 77.47)
+			(xy 119.38 85.09) (xy 130.81 85.09)
 		)
 		(stroke
@@
 	(wire
 		(pts
-			(xy 201.93 110.49) (xy 201.93 121.92)
+			(xy 201.93 58.42) (xy 201.93 77.47)
 		)
 		(stroke
@@
 	(wire
 		(pts
-			(xy 165.1 180.34) (xy 165.1 184.15)
+			(xy 201.93 110.49) (xy 201.93 121.92)
 		)
 		(stroke
@@
 	(wire
 		(pts
-			(xy 135.89 118.11) (xy 142.24 118.11)
+			(xy 165.1 180.34) (xy 165.1 184.15)
 		)
 		(stroke
@@
 	(wire
 		(pts
-			(xy 97.79 184.15) (xy 97.79 161.29)
-		)
-		(stroke
-			(width 0)
-			(type default)
-		)
-	)
-	(wire
-		(pts
 			(xy 177.8 66.04) (xy 189.23 66.04)
 		)
@@
 	(wire
 		(pts
+			(xy 273.05 204.47) (xy 273.05 179.07)
+		)
+		(stroke
+			(width 0)
+			(type default)
+		)
+	)
+	(wire
+		(pts
 			(xy 269.24 66.04) (xy 269.24 156.21)
 		)
@@
 	(wire
 		(pts
+			(xy 147.32 189.23) (xy 147.32 204.47)
+		)
+		(stroke
+			(width 0)
+			(type default)
+		)
+	)
+	(wire
+		(pts
 			(xy 264.16 87.63) (xy 229.87 87.63)
 		)
@@
 	(wire
 		(pts
-			(xy 147.32 184.15) (xy 97.79 184.15)
-		)
-		(stroke
-			(width 0)
-			(type default)
-		)
-	)
-	(wire
-		(pts
 			(xy 40.64 40.64) (xy 40.64 58.42)
 		)
@@
 	(wire
 		(pts
+			(xy 146.05 184.15) (xy 147.32 184.15)
+		)
+		(stroke
+			(width 0)
+			(type default)
+		)
+	)
+	(wire
+		(pts
 			(xy 156.21 40.64) (xy 156.21 58.42)
 		)
@@
 	(wire
 		(pts
-			(xy 119.38 118.11) (xy 135.89 118.11)
+			(xy 119.38 118.11) (xy 142.24 118.11)
 		)
 		(stroke
@@
 					(unit 1)
 				)
-			)
-		)
-	)
-	(symbol
-		(lib_id "Diode:1N4148")
-		(at 135.89 121.92 270)
-		(unit 1)
-		(body_style 1)
-		(exclude_from_sim no)
-		(in_bom yes)
-		(on_board yes)
-		(in_pos_files yes)
-		(dnp no)
-		(fields_autoplaced yes)
-		(property "Reference" "D83"
-			(at 138.43 120.6499 90)
-			(show_name no)
-			(do_not_autoplace no)
-			(effects
-				(font
-					(size 1.27 1.27)
-				)
-				(justify left)
-			)
-		)
-		(property "Value" "1N4148"
-			(at 138.43 123.1899 90)
-			(show_name no)
-			(do_not_autoplace no)
-			(effects
-				(font
-					(size 1.27 1.27)
-				)
-				(justify left)
-			)
-		)
-		(property "Footprint" "Diode_THT:D_DO-35_SOD27_P7.62mm_Horizontal"
-			(at 135.89 121.92 0)
-			(hide yes)
-			(show_name no)
-			(do_not_autoplace no)
-			(effects
-				(font
-					(size 1.27 1.27)
-				)
-			)
-		)
-		(property "Datasheet" "https://assets.nexperia.com/documents/data-sheet/1N4148_1N4448.pdf"
-			(at 135.89 121.92 0)
-			(hide yes)
-			(show_name no)
-			(do_not_autoplace no)
-			(effects
-				(font
-					(size 1.27 1.27)
-				)
-			)
-		)
-		(property "Description" "100V 0.15A standard switching diode, DO-35"
-			(at 135.89 121.92 0)
-			(hide yes)
-			(show_name no)
-			(do_not_autoplace no)
-			(effects
-				(font
-					(size 1.27 1.27)
-				)
-			)
-		)
-		(property "Sim.Device" "D"
-			(at 135.89 121.92 0)
-			(hide yes)
-			(show_name no)
-			(do_not_autoplace no)
-			(effects
-				(font
-					(size 1.27 1.27)
-				)
-			)
-		)
-		(property "Sim.Pins" "1=K 2=A"
-			(at 135.89 121.92 0)
-			(hide yes)
-			(show_name no)
-			(do_not_autoplace no)
-			(effects
-				(font
-					(size 1.27 1.27)
-				)
-			)
-		)
-		(pin "1"
-		)
-		(pin "2"
-		)
-		(instances
-			(project "keyboard"
-				(path "/026a5706-fdc0-4427-9d80-94609c064bdd"
-					(reference "D83")
-					(unit 1)
-				)
